Commit message: spherical joint + fixed based

File: rsc/kinova/urdf/kinova_no_fingers.urdf (robot description, URDF)
Before this commit: robot kinova, 10 links, 9 joints
Joints:
- joint kinova_joint_5: limit lower=-6.28318530718 upper=62.8318530718 effort=6.8 velocity=15 -> lower=0.0 upper=62.8318530718 effort=6.8 velocity=15; type revolute -> spherical

Commit message: final done

File: rsc/kinova/urdf/kinova_no_fingers.urdf (robot description, URDF)
Before this commit: robot kinova, 10 links, 9 joints
Joints:
- joint kinova_joint_5: type spherical -> revolute
